File: eV-LTZ.sch (KiCad schematic (older format))
At the start: 35 parts, among them P1 VIN+, P2 CONN_01X02, P3 VH-, P4 VH+, P5 SENSE-, P6 SENSE+, P7 VIN-, Q1 BD139, U1 LT1013N8

Commit message: modify layout
Connections:
- net labels added: CURRENT_OUT, HEATER+, HEATER-, TCOMP, TSENSE_B, TSENSE_C, VCC, ZENER-
- net labels removed: TSENSE
- wire segments 87 -> 83
Changed lines of the file:
@@
 LIBS:sensors
 LIBS:lp2951
+LIBS:eV-LTZ-cache
 EELAYER 25 0
 EELAYER END
@@
 Wire Wire Line
 	2500 1475 5375 1475
-Wire Wire Line
-	1650 4350 1650 3275
 Connection ~ 1650 4350
 Wire Wire Line
@@
 Wire Wire Line
 	1525 1675 2575 1675
-Wire Wire Line
-	1650 1475 1650 2975
 Connection ~ 1650 1475
-Wire Wire Line
-	1900 1675 1900 2975
 Connection ~ 1900 1675
 Connection ~ 10100 1925
@@
 Text Label 1525 1675 0    60   ~ 0
 VH+
-Wire Wire Line
-	1900 3275 1900 4100
 Connection ~ 1900 4100
 Text Label 1400 4100 0    60   ~ 0
@@
 HEAT
 Text Label 6725 2475 2    60   ~ 0
-TSENSE
+TSENSE_B
 Text Label 1075 3750 0    60   ~ 0
 VIN-
@@
 Wire Wire Line
 	3050 1475 3050 3125
+Text Label 8250 2100 0    60   ~ 0
+TCOMP
+Text Label 7725 3225 0    60   ~ 0
+ZENER-
+Text Label 9625 2375 0    60   ~ 0
+CURRENT_OUT
+Text Label 6300 2100 0    60   ~ 0
+TSENSE_C
+Text Label 4000 2975 0    60   ~ 0
+HEATER+
+Text Label 3275 1675 0    60   ~ 0
+VCC
+Text Label 3975 4100 0    60   ~ 0
+HEATER-
 $EndSCHEMATC
