File: eV-LTZ.sch (KiCad schematic (older format))
At the start: 35 parts, among them P1 VIN+, P2 CONN_01X02, P3 VH-, P4 VH+, P5 SENSE-, P6 SENSE+, P7 VIN-, Q1 BD139, U1 LT1013N8

Commit message: improve traces
Parts:
- added R4.2: 25k, Resistors_THT:R_Axial_DIN0617_L17.0mm_D6.0mm_P20.32mm_Horizontal, symbol R
- C10, C5: footprint Capacitors_THT:CP_Radial_Tantal_D5.0mm_P5.00mm -> Capacitors_THT:CP_Radial_D8.0mm_P5.00mm
- P2: value CONN_01X02 -> TEMP NTC; footprint Connectors:bornier2 -> Connectors_Samtec:SL-102-X-XX_1x02
- P5, P6: footprint Connectors:1pin -> Measurement_Points:Measurement_Point_Round-TH_Big
- R4.1: value 12k -> 25k
Connections:
- net labels added: VCCH, VCCOPAMP
- net labels removed: VCC
- wire segments 83 -> 86
